Commit message: [Twin Hammer] [urdf] [control] Changed mass of main body due to change the cables of real machine changed the gravity comp in controller

File: robots/twin_hammer/urdf/device.urdf.xacro (robot description, xacro)
@@ -291,5 +291,5 @@
  <link name="main_body">
    <inertial>
-     <mass value = "0.25" />
+     <mass value = "1.2" />
      <origin xyz="0.1356 -0.0001 -0.0139" rpy="0 0 0"/>
      <inertia

File: robots/twin_hammer/urdf/device_with_dummy_weight.urdf.xacro (robot description, xacro)
@@ -291,5 +291,5 @@
  <link name="main_body">
    <inertial>
-     <mass value = "0.25" />
+     <mass value = "1.2" />
      <origin xyz="0.1356 -0.0001 -0.0139" rpy="0 0 0"/>
      <inertia
