Commit message: [gimbalrotor] [beetle_kaneko] Change servo.yaml and config in spinal from kondo to dynamixel change beetle urdf

File: robots/gimbalrotor/urdf/beetle/gimbalrotor.urdf.xacro (robot description, xacro)
@@ -23,10 +23,10 @@
     <link name="base_link">
       <inertial>
-        <origin xyz="0.000169 0.002346 0.106123" rpy="0 0 0"/>
-        <mass value="1.37825"/>
-        <inertia
-            ixx="0.046756" ixy="0.000586" ixz="0.000055"
-	    iyy="0.063216" iyz="0.000219"
-	    izz="0.058783"/>
+        <origin xyz="0.013574 0.001135 0.041962" rpy="0 0 0"/>
+        <mass value="1.20490"/>
+        <inertia
+            ixx="0.010610" ixy="-0.000085" ixz="0.000340"
+            iyy="0.020290" iyz="0.000116"
+            izz="0.021260"/>
       </inertial>
       <visual>
@@ -82,8 +82,8 @@
     </xacro:macro>
     ## dummy rotor arms
-    <xacro:dummy_rotor_arm id = "${child1}" x = "0.12129" y="0.12150" z = "0.1185" yaw = "${pi/4.0}"/>
-    <xacro:dummy_rotor_arm id = "${child2}" x = "-0.12129" y="0.12150" z = "0.1185" yaw = "${pi*3.0/4.0}"/>
-    <xacro:dummy_rotor_arm id = "${child3}" x = "-0.12129" y="-0.12150" z = "0.1185" yaw = "${pi*5.0/4.0}"/>
-    <xacro:dummy_rotor_arm id = "${child4}" x = "0.12129" y="-0.12150" z = "0.1185" yaw = "${-pi/4.0}"/>
+    <xacro:dummy_rotor_arm id = "${child1}" x = "0.15410" y="0.15424" z = "0.1185" yaw = "${pi/4.0}"/>
+    <xacro:dummy_rotor_arm id = "${child2}" x = "-0.15410" y="0.15424" z = "0.1185" yaw = "${pi*3.0/4.0}"/>
+    <xacro:dummy_rotor_arm id = "${child3}" x = "-0.15410" y="-0.15424" z = "0.1185" yaw = "${pi*5.0/4.0}"/>
+    <xacro:dummy_rotor_arm id = "${child4}" x = "0.15410" y="-0.15424" z = "0.1185" yaw = "${-pi/4.0}"/>
     ## dummy link for the contact point coordinate
       <link name="contact_point">

Commit message: [gimbalrotor] [beetle_kaneko] some modification around urdf and motorinfo based on real machine exp

File: robots/gimbalrotor/urdf/beetle/gimbalrotor.urdf.xacro (robot description, xacro)
@@ -23,5 +23,5 @@
     <link name="base_link">
       <inertial>
-        <origin xyz="0.013574 0.001135 0.041962" rpy="0 0 0"/>
+        <origin xyz="0.004 0.001135 0.041962" rpy="0 0 0"/>
         <mass value="1.20490"/>
         <inertia
