Commit message: [Dracomancer] dracomancer.xacroを人間上肢に

File: robots/dracomancer/urdf/dracomancer.xacro (robot description, xacro)
@@ -1,9 +1,88 @@
 <?xml version="1.0"?>
-<robot name="exoskeleton" xmlns:xacro="http://www.ros.org/wiki/xacro">
-  <!-- パラメータ -->
+<robot name="human_arm_7dof" xmlns:xacro="http://www.ros.org/wiki/xacro">
+  <!-- ===== Parameters ===== -->
+  <xacro:property name="pi" value="3.141592653589793"/>
+  <!-- Lengths [m] -->
   <xacro:property name="upper_arm_length" value="0.30"/>
-  <xacro:property name="forearm_length" value="0.25"/>
-  <xacro:property name="hand_length" value="0.12"/>
-  <!-- 材質 -->
+  <xacro:property name="forearm_length"  value="0.25"/>
+  <xacro:property name="hand_length"     value="0.12"/>
+  <!-- Radii [m] -->
+  <xacro:property name="upper_arm_radius" value="0.04"/>
+  <xacro:property name="forearm_radius"   value="0.035"/>
+  <xacro:property name="wrist_radius"     value="0.03"/>
+  <!-- Masses [kg] -->
+  <xacro:property name="upper_arm_mass" value="2.0"/>
+  <xacro:property name="forearm_mass"   value="1.5"/>
+  <xacro:property name="hand_mass"      value="0.6"/>
+  <!-- ===== Macros ===== -->
+  <xacro:macro name="box_inertial" params="mass x y z">
+    <inertial>
+      <mass value="${mass}"/>
+      <origin xyz="0 0 0" rpy="0 0 0"/>
+      <inertia
+        ixx="${mass*(y*y+z*z)/12.0}"
+        ixy="0.0"
+        ixz="0.0"
+        iyy="${mass*(x*x+z*z)/12.0}"
+        iyz="0.0"
+        izz="${mass*(x*x+y*y)/12.0}"/>
+    </inertial>
+  </xacro:macro>
+  <xacro:macro name="cylinder_inertial" params="mass radius length axis">
+    <inertial>
+      <mass value="${mass}"/>
+      <origin xyz="0 0 0" rpy="0 0 0"/>
+      <!-- default: cylinder whose principal axis is z -->
+      <xacro:if value="${axis == 'z'}">
+        <inertia
+          ixx="${mass*(3*radius*radius + length*length)/12.0}"
+          ixy="0.0"
+          ixz="0.0"
+          iyy="${mass*(3*radius*radius + length*length)/12.0}"
+          iyz="0.0"
+          izz="${0.5*mass*radius*radius}"/>
+      </xacro:if>
+      <!-- cylinder principal axis is x -->
+      <xacro:if value="${axis == 'x'}">
+        <inertia
+          ixx="${0.5*mass*radius*radius}"
+          ixy="0.0"
+          ixz="0.0"
+          iyy="${mass*(3*radius*radius + length*length)/12.0}"
+          iyz="0.0"
+          izz="${mass*(3*radius*radius + length*length)/12.0}"/>
+      </xacro:if>
+      <!-- cylinder principal axis is y -->
+      <xacro:if value="${axis == 'y'}">
+        <inertia
+          ixx="${mass*(3*radius*radius + length*length)/12.0}"
+          ixy="0.0"
+          ixz="0.0"
+          iyy="${0.5*mass*radius*radius}"
+          iyz="0.0"
+          izz="${mass*(3*radius*radius + length*length)/12.0}"/>
+      </xacro:if>
+    </inertial>
+  </xacro:macro>
+  <xacro:macro name="arm_segment" params="name length radius mass color">
+    <link name="${name}">
+      <visual>
+        <!-- cylinder axis is z, so rotate to align along x -->
+        <origin xyz="${length/2.0} 0 0" rpy="0 ${pi/2.0} 0"/>
+        <geometry>
+          <cylinder radius="${radius}" length="${length}"/>
+        </geometry>
+        <material name="${color}"/>
+      </visual>
+      <collision>
+        <origin xyz="${length/2.0} 0 0" rpy="0 ${pi/2.0} 0"/>
+        <geometry>
+          <cylinder radius="${radius}" length="${length}"/>
+        </geometry>
+      </collision>
+      <xacro:cylinder_inertial mass="${mass}" radius="${radius}" length="${length}" axis="x"/>
+    </link>
+  </xacro:macro>
+  <!-- ===== Materials ===== -->
   <material name="gray">
     <color rgba="0.7 0.7 0.7 1.0"/>
@@ -12,95 +91,130 @@
     <color rgba="0.2 0.4 0.9 1.0"/>
   </material>
-  <!-- base -->
-  <link name="base_link">
+  <material name="green">
+    <color rgba="0.2 0.8 0.3 1.0"/>
+  </material>
+  <material name="orange">
+    <color rgba="0.95 0.55 0.15 1.0"/>
+  </material>
+  <!-- ===== Base ===== -->
+  <link name="torso_anchor">
     <visual>
-      <geometry>
-        <box size="0.08 0.08 0.08"/>
+      <origin xyz="0 0 0" rpy="0 0 0"/>
+      <geometry>
+        <box size="0.12 0.12 0.12"/>
       </geometry>
       <material name="gray"/>
     </visual>
+    <collision>
+      <origin xyz="0 0 0" rpy="0 0 0"/>
+      <geometry>
+        <box size="0.12 0.12 0.12"/>
+      </geometry>
+    </collision>
+    <xacro:box_inertial mass="5.0" x="0.12" y="0.12" z="0.12"/>
   </link>
-  <!-- shoulder yaw -->
-  <link name="shoulder_yaw_link">
+  <!-- dummy links for multi-DoF shoulder -->
+  <link name="shoulder_yaw_link"/>
+  <link name="shoulder_pitch_link"/>
+  <link name="shoulder_roll_link"/>
+  <link name="elbow_link"/>
+  <link name="forearm_rot_link"/>
+  <link name="wrist_pitch_link"/>
+  <link name="wrist_yaw_link"/>
+  <!-- actual geometry links -->
+  <xacro:arm_segment name="upper_arm_link"
+                     length="${upper_arm_length}"
+                     radius="${upper_arm_radius}"
+                     mass="${upper_arm_mass}"
+                     color="blue"/>
+  <xacro:arm_segment name="forearm_link"
+                     length="${forearm_length}"
+                     radius="${forearm_radius}"
+                     mass="${forearm_mass}"
+                     color="green"/>
+  <link name="hand_link">
     <visual>
-      <geometry>
-        <cylinder radius="0.03" length="0.08"/>
-      </geometry>
-      <material name="blue"/>
+      <origin xyz="${hand_length/2.0} 0 0" rpy="0 0 0"/>
+      <geometry>
+        <box size="${hand_length} 0.06 0.025"/>
+      </geometry>
+      <material name="orange"/>
     </visual>
+    <collision>
+      <origin xyz="${hand_length/2.0} 0 0" rpy="0 0 0"/>
+      <geometry>
+        <box size="${hand_length} 0.06 0.025"/>
+      </geometry>
+    </collision>
+    <xacro:box_inertial mass="${hand_mass}" x="${hand_length}" y="0.06" z="0.025"/>
   </link>
-  <joint name="shoulder_yaw" type="revolute">
-    <parent link="base_link"/>
+  <!-- ===== Joints ===== -->
+  <!-- Shoulder 3DoF -->
+  <joint name="shoulder_yaw_joint" type="revolute">
+    <parent link="torso_anchor"/>
     <child link="shoulder_yaw_link"/>
-    <origin xyz="0 0 0.05" rpy="0 0 0"/>
+    <origin xyz="0 0.10 0" rpy="0 0 0"/>
     <axis xyz="0 0 1"/>
-    <limit lower="-3.14" upper="3.14" effort="10" velocity="2.0"/>
-  </joint>
-  <!-- shoulder pitch -->
-  <link name="shoulder_pitch_link">
-    <visual>
-      <geometry>
-        <cylinder radius="0.025" length="0.08"/>
-      </geometry>
-      <material name="blue"/>
-    </visual>
-  </link>
-  <joint name="shoulder_pitch" type="revolute">
+    <limit lower="${-pi}" upper="${pi}" effort="30" velocity="3.0"/>
+  </joint>
+  <joint name="shoulder_pitch_joint" type="revolute">
     <parent link="shoulder_yaw_link"/>
     <child link="shoulder_pitch_link"/>
-    <origin xyz="0 0 0.04" rpy="0 1.5708 0"/>
+    <origin xyz="0 0 0" rpy="0 0 0"/>
     <axis xyz="0 1 0"/>
-    <limit lower="-1.57" upper="1.57" effort="10" velocity="2.0"/>
-  </joint>
-  <!-- upper arm -->
-  <link name="upper_arm_link">
-    <visual>
-      <origin xyz="0 0 -${upper_arm_length/2}" rpy="0 0 0"/>
-      <geometry>
-        <cylinder radius="0.02" length="${upper_arm_length}"/>
-      </geometry>
-      <material name="gray"/>
-    </visual>
-  </link>
-  <joint name="shoulder_roll" type="revolute">
+    <limit lower="${-pi/2.0}" upper="${pi/2.0}" effort="30" velocity="3.0"/>
+  </joint>
+  <joint name="shoulder_roll_joint" type="revolute">
     <parent link="shoulder_pitch_link"/>
+    <child link="shoulder_roll_link"/>
+    <origin xyz="0 0 0" rpy="0 0 0"/>
+    <axis xyz="1 0 0"/>
+    <limit lower="${-pi/2.0}" upper="${pi/2.0}" effort="20" velocity="3.0"/>
+  </joint>
+  <joint name="upper_arm_fixed" type="fixed">
+    <parent link="shoulder_roll_link"/>
     <child link="upper_arm_link"/>
-    <origin xyz="0 0 0.04" rpy="0 0 0"/>
+    <origin xyz="0 0 0" rpy="0 0 0"/>
+  </joint>
+  <!-- Elbow flexion -->
+  <joint name="elbow_flex_joint" type="revolute">
+    <parent link="upper_arm_link"/>
+    <child link="elbow_link"/>
+    <origin xyz="${upper_arm_length} 0 0" rpy="0 0 0"/>
+    <axis xyz="0 1 0"/>
+    <limit lower="0.0" upper="${5.0*pi/6.0}" effort="20" velocity="3.0"/>
+  </joint>
+  <joint name="forearm_fixed" type="fixed">
+    <parent link="elbow_link"/>
+    <child link="forearm_rot_link"/>
+    <origin xyz="0 0 0" rpy="0 0 0"/>
+  </joint>
+  <!-- Forearm pronation/supination -->
+  <joint name="forearm_rot_joint" type="revolute">
+    <parent link="forearm_rot_link"/>
+    <child link="forearm_link"/>
+    <origin xyz="0 0 0" rpy="0 0 0"/>
     <axis xyz="1 0 0"/>
-    <limit lower="-1.57" upper="1.57" effort="10" velocity="2.0"/>
-  </joint>
-  <!-- forearm -->
-  <link name="forearm_link">
-    <visual>
-      <origin xyz="0 0 -${forearm_length/2}" rpy="0 0 0"/>
-      <geometry>
-        <cylinder radius="0.018" length="${forearm_length}"/>
-      </geometry>
-      <material name="gray"/>
-    </visual>
-  </link>
-  <joint name="elbow_flex" type="revolute">
-    <parent link="upper_arm_link"/>
-    <child link="forearm_link"/>
-    <origin xyz="0 0 -${upper_arm_length}" rpy="0 0 0"/>
+    <limit lower="${-pi}" upper="${pi}" effort="10" velocity="4.0"/>
+  </joint>
+  <!-- Wrist 2DoF -->
+  <joint name="wrist_pitch_joint" type="revolute">
+    <parent link="forearm_link"/>
+    <child link="wrist_pitch_link"/>
+    <origin xyz="${forearm_length} 0 0" rpy="0 0 0"/>
     <axis xyz="0 1 0"/>
-    <limit lower="0.0" upper="2.6" effort="10" velocity="2.0"/>
-  </joint>
-  <!-- hand -->
-  <link name="hand_link">
-    <visual>
-      <origin xyz="0 0 -${hand_length/2}" rpy="0 0 0"/>
-      <geometry>
-        <box size="0.05 0.03 ${hand_length}"/>
-      </geometry>
-      <material name="blue"/>
-    </visual>
-  </link>
-  <joint name="wrist_pitch" type="revolute">
-    <parent link="forearm_link"/>
+    <limit lower="${-pi/2.0}" upper="${pi/2.0}" effort="8" velocity="4.0"/>
+  </joint>
+  <joint name="wrist_yaw_joint" type="revolute">
+    <parent link="wrist_pitch_link"/>
+    <child link="wrist_yaw_link"/>
+    <origin xyz="0 0 0" rpy="0 0 0"/>
+    <axis xyz="0 0 1"/>
+    <limit lower="${-pi/2.0}" upper="${pi/2.0}" effort="8" velocity="4.0"/>
+  </joint>
+  <joint name="hand_fixed" type="fixed">
+    <parent link="wrist_yaw_link"/>
     <child link="hand_link"/>
-    <origin xyz="0 0 -${forearm_length}" rpy="0 0 0"/>
-    <axis xyz="0 1 0"/>
-    <limit lower="-1.0" upper="1.0" effort="10" velocity="2.0"/>
+    <origin xyz="0 0 0" rpy="0 0 0"/>
   </joint>
 </robot>
