Commit message: [Dracomancer] xacroファイルを改名，stlファイルのパスを修正

File: robots/dracomancer/urdf/dracomancer.urdf (robot description, URDF)
Before this commit: robot dracomancer, 8 links, 7 joints
Links:
- link base_link: geometry collision mesh filename=package://dracomancer/urdf/mesh/base.STL scale=0.001 0.001 0.001; visual mesh filename=package://dracomancer/urdf/mesh/base.STL scale=0.001 0.001 0.001
- link hand_link: geometry collision mesh filename=package://dracomancer/urdf/mesh/hand.STL scale=0.001 0.001 0.001; visual mesh filename=package://dracomancer/urdf/mesh/hand.STL scale=0.001 0.001 0.001
- link lower_arm_lower_link: geometry collision mesh filename=package://dracomancer/urdf/mesh/lower_arm_lower.STL scale=0.001 0.001 0.001; visual mesh filename=package://dracomancer/urdf/mesh/lower_arm_lower.STL scale=0.001 0.001 0.001
- link lower_arm_upper_link: geometry collision mesh filename=package://dracomancer/urdf/mesh/lower_arm_upper.STL scale=0.001 0.001 0.001; visual mesh filename=package://dracomancer/urdf/mesh/lower_arm_upper.STL scale=0.001 0.001 0.001
- link shoulder_link: geometry collision mesh filename=package://dracomancer/urdf/mesh/shoulder.STL scale=0.001 0.001 0.001; visual mesh filename=package://dracomancer/urdf/mesh/shoulder.STL scale=0.001 0.001 0.001
- link upper_arm_lower_link: geometry collision mesh filename=package://dracomancer/urdf/mesh/upper_arm_lower.STL scale=0.001 0.001 0.001; visual mesh filename=package://dracomancer/urdf/mesh/upper_arm_lower.STL scale=0.001 0.001 0.001
- link upper_arm_upper_link: geometry collision mesh filename=package://dracomancer/urdf/mesh/upper_arm_upper.STL scale=0.001 0.001 0.001; visual mesh filename=package://dracomancer/urdf/mesh/upper_arm_upper.STL scale=0.001 0.001 0.001
- link wrist_link: geometry collision mesh filename=package://dracomancer/urdf/mesh/wrist.STL scale=0.001 0.001 0.001; visual mesh filename=package://dracomancer/urdf/mesh/wrist.STL scale=0.001 0.001 0.001

File: robots/dracomancer/urdf/human_arm.xacro (robot description, xacro)
@@ -1,4 +1,4 @@
 <?xml version="1.0"?>
-<robot name="dracomancer" xmlns:xacro="http://www.ros.org/wiki/xacro">
+<robot name="human_arm" xmlns:xacro="http://www.ros.org/wiki/xacro">
   <!-- ===== Parameters ===== -->
   <xacro:property name="pi" value="3.141592653589793"/>

Commit message: [Dracomancer] urdfの結合を記述

File: robots/dracomancer/urdf/dracomancer.urdf (robot description, URDF)
Before this commit: robot dracomancer, 8 links, 7 joints
Joints:
- removed joint elbow_joint
- removed joint hand_joint
- removed joint lower_arm_lower_joint
- removed joint shoulder_joint
- removed joint upper_arm_lower_joint
- removed joint upper_arm_upper_joint
- removed joint wrist_joint
- added joint elbow_flexion_extension_joint: type revolute, parent upper_arm_lower_link, child lower_arm_upper_link, origin xyz=0.20 0.00 0.00 rpy=0 0 0, axis 1 0 0, limit lower=0.0 upper=2.4 effort=20 velocity=2.0
- added joint shoulder_abduction_adduction_joint: type revolute, parent base_link, child shoulder_link, origin xyz=0.00 0.00 0.00 rpy=0 0 0, axis 0 1 0, limit lower=-1.57 upper=1.57 effort=30 velocity=2.0
- added joint shoulder_flexion_extension_joint: type revolute, parent shoulder_link, child upper_arm_upper_link, origin xyz=0.00 0.00 0.00 rpy=0 0 0, axis 1 0 0, limit lower=-1.57 upper=1.57 effort=30 velocity=2.0
- added joint upper_arm_external_internal_rotation_joint: type revolute, parent upper_arm_upper_link, child upper_arm_lower_link, origin xyz=0.03 0.00 0.00 rpy=0 0 0, axis 0 0 1, limit lower=-1.57 upper=1.57 effort=30 velocity=2.0
- added joint wrist_abduction_adduction_joint: type revolute, parent wrist_link, child hand_link, origin xyz=0.18 0.00 0.00 rpy=0 0 0, axis 0 1 0, limit lower=-1.0 upper=1.0 effort=10 velocity=2.0
- added joint wrist_flexion_extension_joint: type revolute, parent lower_arm_lower_link, child wrist_link, origin xyz=0.18 0.00 0.00 rpy=0 0 0, axis 1 0 0, limit lower=-1.57 upper=1.57 effort=10 velocity=2.0
- added joint wrist_supination_joint: type revolute, parent lower_arm_upper_link, child lower_arm_lower_link, origin xyz=0.20 0.00 0.00 rpy=0 0 0, axis 0 0 1, limit lower=0.0 upper=2.4 effort=20 velocity=2.0

Commit message: [Dracomancer] URDFのorigin位置を0 0 0 に設定

File: robots/dracomancer/urdf/dracomancer.urdf (robot description, URDF)
Before this commit: robot dracomancer, 8 links, 7 joints
Joints:
- joint elbow_flexion_extension_joint: origin xyz=0.20 0.00 0.00 rpy=0 0 0 -> xyz=0.00 0.00 0.00 rpy=0 0 0
- joint upper_arm_external_internal_rotation_joint: origin xyz=0.03 0.00 0.00 rpy=0 0 0 -> xyz=0.00 0.00 0.00 rpy=0 0 0
- joint wrist_abduction_adduction_joint: origin xyz=0.18 0.00 0.00 rpy=0 0 0 -> xyz=0.00 0.00 0.00 rpy=0 0 0
- joint wrist_flexion_extension_joint: origin xyz=0.18 0.00 0.00 rpy=0 0 0 -> xyz=0.00 0.00 0.00 rpy=0 0 0
- joint wrist_supination_joint: origin xyz=0.20 0.00 0.00 rpy=0 0 0 -> xyz=0.00 0.00 0.00 rpy=0 0 0

Commit message: [Dracomancer] bringup.launchからjoint_state_publisher_guiを削除し，ジョイント位置を決定

File: robots/dracomancer/urdf/dracomancer.urdf (robot description, URDF)
Before this commit: robot dracomancer, 8 links, 7 joints
Joints:
- joint elbow_flexion_extension_joint: origin xyz=0.00 0.00 0.00 rpy=0 0 0 -> xyz=-0.00675 0.00 -0.1209 rpy=0 0 0
- joint shoulder_flexion_extension_joint: origin xyz=0.00 0.00 0.00 rpy=0 0 0 -> xyz=0.0925 0.001 -0.1025 rpy=0 0 0
- joint upper_arm_external_internal_rotation_joint: origin xyz=0.00 0.00 0.00 rpy=0 0 0 -> xyz=-0.0209 0.00 -0.09475 rpy=0 0 0
- joint wrist_abduction_adduction_joint: origin xyz=0.00 0.00 0.00 rpy=0 0 0 -> xyz=-0.03915 0.0209 -0.0225 rpy=0 0 0
- joint wrist_flexion_extension_joint: origin xyz=0.00 0.00 0.00 rpy=0 0 0 -> xyz=-0.00675 0.00 -0.1209 rpy=0 0 0
- joint wrist_supination_joint: origin xyz=0.00 0.00 0.00 rpy=0 0 0 -> xyz=-0.0209 0.00 -0.09475 rpy=0 0 0

Commit message: [Dracomancer] ロボットをz方向に1mオフセット

File: robots/dracomancer/urdf/dracomancer.urdf (robot description, URDF)
Before this commit: robot dracomancer, 9 links, 8 joints
Joints:
- joint world_to_base: origin xyz=0.00 0.00 0.00 rpy=0 0 0 -> xyz=0.00 0.00 1.00 rpy=0 0 0

Commit message: [Dracomancer] upper_link_upperまでinertial追加

File: robots/dracomancer/urdf/dracomancer.urdf (robot description, URDF)
Before this commit: robot dracomancer, 9 links, 8 joints
Links:
- link base_link: mass 3.0 -> None
- link shoulder_link: mass 1.0 -> 0.09741
- link upper_arm_upper_link: mass 0.8 -> 0.09741

Commit message: [Dracomancer] URDFに物理パラメータを入力

File: robots/dracomancer/urdf/dracomancer.urdf (robot description, URDF)
Before this commit: robot dracomancer, 9 links, 8 joints
Links:
- link base_link: mass None -> 0.1
- link hand_link: mass 0.3 -> 0.23533
- link lower_arm_lower_link: mass 0.7 -> 0.11630
- link lower_arm_upper_link: mass 0.7 -> 0.09741
- link upper_arm_lower_link: mass 0.8 -> 0.11630
- link wrist_link: mass 0.4 -> 0.06312
Joints:
- joint elbow_flexion_extension_joint: limit lower=0.0 upper=2.4 effort=20 velocity=2.0 -> lower=-1.57 upper=1.57 effort=0.4 velocity=1.0
- joint shoulder_abduction_adduction_joint: limit lower=-1.57 upper=1.57 effort=30 velocity=2.0 -> lower=-1.57 upper=1.57 effort=0.4 velocity=1.0
- joint shoulder_flexion_extension_joint: limit lower=-1.57 upper=1.57 effort=30 velocity=2.0 -> lower=-1.57 upper=1.57 effort=0.4 velocity=1.0
- joint upper_arm_external_internal_rotation_joint: limit lower=-1.57 upper=1.57 effort=30 velocity=2.0 -> lower=-1.57 upper=1.57 effort=0.4 velocity=1.0
- joint wrist_abduction_adduction_joint: limit lower=-1.0 upper=1.0 effort=10 velocity=2.0 -> lower=-1.57 upper=1.57 effort=0.4 velocity=1.0
- joint wrist_flexion_extension_joint: limit lower=-1.57 upper=1.57 effort=10 velocity=2.0 -> lower=-1.57 upper=1.57 effort=0.4 velocity=1.0
- joint wrist_supination_joint: limit lower=0.0 upper=2.4 effort=20 velocity=2.0 -> lower=-1.57 upper=1.57 effort=0.4 velocity=1.0

Commit message: [Dracomancer] control_joints.pyを修正

File: robots/dracomancer/urdf/dracomancer.urdf (robot description, URDF)
Before this commit: robot dracomancer, 9 links, 8 joints
Links:
- link base_link: mass 0.1 -> 0.92761

Commit message: [Dracomancer] fix: サーボ回転方向を修正

File: robots/dracomancer/urdf/dracomancer.urdf (robot description, URDF)
Before this commit: robot dracomancer, 9 links, 8 joints
Joints:
- joint elbow_flexion_extension_joint: axis 1 0 0 -> -1 0 0
- joint shoulder_flexion_extension_joint: axis 1 0 0 -> -1 0 0
- joint wrist_flexion_extension_joint: axis 1 0 0 -> -1 0 0

Commit message: [Dracomancer] URDF・回転方向を修正

File: robots/dracomancer/urdf/dracomancer.urdf (robot description, URDF)
Before this commit: robot dracomancer, 9 links, 8 joints
Joints:
- joint wrist_supination_joint: axis 0 0 1 -> 0 0 -1

Commit message: [Dracomancer] 修正

File: robots/dracomancer/urdf/dracomancer.urdf (robot description, URDF)
Before this commit: robot dracomancer, 9 links, 8 joints
Joints:
- joint upper_arm_external_internal_rotation_joint: axis 0 0 1 -> 0 0 -1
